File: IMU.kicad_sch (KiCad schematic)
At the start: 25 parts, among them J1 USB_B_Micro, J2 Conn_01x10_MountingPin, J3 Conn_01x04_MountingPin, J5 Conn_01x04_MountingPin, J7 Conn_02x03_Counter_Clockwise, U2 HT75xx-1-SOT89, U3 ISM330DLCTR, U4 STM32F401RCT6TR

Commit message: first draft
Other:
- note added: "IMU Sensor with STM32"
- note added: "Nithya Sudharshan"
Changed lines of the file:
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@@
+		)
+	)
+	(text "IMU Sensor with STM32"
+		(exclude_from_sim no)
+		(at 210.058 189.738 0)
+		(effects
+			(font
+				(size 2.54 2.54)
+				(thickness 0.254)
+				(bold yes)
+			)
 		)
 	)
@@
 			)
 		)
+	)
+	(text "Nithya Sudharshan"
+		(exclude_from_sim no)
+		(at 197.104 183.388 0)
+		(effects
+			(font
+				(size 1.27 1.27)
+				(thickness 0.254)
+				(bold yes)
+			)
+		)
