File: hardware/IMU.kicad_sch (KiCad schematic)
At the start: 37 parts, among them J2 Conn_01x09, J3 USB_B_Micro, J4 Conn_01x10, J6 Conn_01x04, J8 Conn_01x04, J9 Conn_01x06, SW1 SW_Push, U2 HT75xx-1-SOT89, U3 ISM330DLCTR, U4 STM32F401RCT6TR, Y2 WE-XTAL_CFPX-104

Commit message: layout first draft
Parts:
- removed J2: Conn_01x09, Connector_PinHeader_2.54mm:PinHeader_1x09_P2.54mm_Vertical, symbol Connector_Generic:Conn_01x09
- added J1: Conn_01x10, Connector_PinHeader_2.54mm:PinHeader_1x10_P2.54mm_Vertical, symbol Connector_Generic:Conn_01x10
- J6: value Conn_01x04 -> UART
- J8: value Conn_01x04 -> IMU_Headers
- J9: value Conn_01x06 -> SWD
- renumbered C12 to C10, C13 to C11, C7 to C12, C15 to C13, C10 to C15, C11 to C16, C16 to C6, C6 to C7
Connections:
- net +3V3: now also D2.2 (A), R1.1; no longer C16.1, R1.2, U2.3 (VOUT)
- net GND: now also J1.1 (Pin_1)
- net RST: now also J9.4 (Pin_4); no longer J9.5 (Pin_5)
- net SWCLK: now also J9.3 (Pin_3); no longer J9.4 (Pin_4)
- net SWDIO: now also J9.5 (Pin_5); no longer J9.3 (Pin_3)
- net at U4.33 (PB12): now also J4.7 (Pin_7); no longer J4.1 (Pin_1)
- net at J4.10 (Pin_10): now also U4.36 (PB15); no longer U4.40 (PC9)
- net at U4.34 (PB13): now also J4.8 (Pin_8); no longer J4.2 (Pin_2)
- net at U4.35 (PB14): now also J4.9 (Pin_9); no longer J4.3 (Pin_3)
- net PA7: now reaches J4.4 (Pin_4)
- net PA7: now also U4.23 (PA7); no longer U4.36 (PB15)
- net PC6: now reaches U4.37 (PC6)
- net PC6: now also J1.10 (Pin_10); no longer J4.7 (Pin_7)
- net PC7: now reaches U4.38 (PC7)
- net PC7: now also J1.9 (Pin_9); no longer J4.8 (Pin_8)
- net PC8: now reaches U4.39 (PC8)
- net PC8: now also J1.8 (Pin_8); no longer J4.9 (Pin_9)
- net at U4.45 (PA12): now also J1.2 (Pin_2)
- net at U4.44 (PA11): now also J1.3 (Pin_3)
- net at U4.43 (PA10): now also J1.4 (Pin_4)
- net at U4.42 (PA9): now also J1.5 (Pin_5)
- net at U4.41 (PA8): now also J1.6 (Pin_6)
- net PA6: now reaches U4.22 (PA6)
- net PA6: now also J4.3 (Pin_3)
- net PA5: now reaches U4.21 (PA5)
- net PA5: now also J4.2 (Pin_2)
- net PA4: now reaches U4.20 (PA4)
- net PA4: now also J4.1 (Pin_1)
- new net: C16.1, R1.2, U2.3 (VOUT)
- new net PC9: J1.7 (Pin_7), U4.40 (PC9)
Other:
- moved on the sheet: C1, J4, R4

Commit message: fixed errors
Changed lines of the file:
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@@
 	(wire
 		(pts
+			(xy 57.15 66.04) (xy 57.15 68.58)
+		)
+		(stroke
+			(width 0)
+			(type default)
+		)
+	)
+	(wire
+		(pts
 			(xy 127 156.21) (xy 130.81 156.21)
 		)
@@
 		)
 	)
+	(label "Vdd"
+		(at 57.15 66.04 0)
+		(effects
+			(font
+				(size 1.27 1.27)
+			)
+			(justify left bottom)
+		)
+	)
 	(label "PA7"
 		(at 135.89 96.52 0)
@@
 					(unit 1)
 				)
-			)
-		)
-	)
-	(symbol
-		(lib_id "power:+3V3")
-		(at 57.15 68.58 0)
-		(unit 1)
-		(exclude_from_sim no)
-		(in_bom yes)
-		(on_board yes)
-		(dnp no)
-		(fields_autoplaced yes)
-		(property "Reference" "#PWR028"
-			(at 57.15 72.39 0)
-			(effects
-				(font
-					(size 1.27 1.27)
-				)
-				(hide yes)
-			)
-		)
-		(property "Value" "+3V3"
-			(at 57.15 63.5 0)
-			(effects
-				(font
-					(size 1.27 1.27)
-				)
-			)
-		)
-		(property "Footprint" ""
-			(at 57.15 68.58 0)
-			(effects
-				(font
-					(size 1.27 1.27)
-				)
-				(hide yes)
-			)
-		)
-		(property "Datasheet" ""
-			(at 57.15 68.58 0)
-			(effects
-				(font
-					(size 1.27 1.27)
-				)
-				(hide yes)
-			)
-		)
-		(property "Description" "Power symbol creates a global label with name \"+3V3\""
-			(at 57.15 68.58 0)
-			(effects
-				(font
-					(size 1.27 1.27)
-				)
-				(hide yes)
-			)
-		)
-		(pin "1"
-		)
-		(instances
-			(project ""
-				(path "/b668f2de-6e3e-4f42-9b63-8394182e1fe8"
-					(reference "#PWR028")
-					(unit 1)
-				)
